Commit message: Add files via upload

File: scr/my_robot_descirption/urdf/mobile_base.xacro (robot description, xacro)
@@ -26,5 +26,5 @@
                            o_xyz = "0 0 ${radius}" o_rpy = "0 0 0"/>
     </link>
-    <link name ="lider_link">
+    <link name ="lidar_link">
         <visual>
             <geometry>
@@ -34,4 +34,12 @@
             <material name = "white"/>
         </visual>
+        <!-- <collision>
+            <geometry>
+                <cylinder radius = "${radius}" length = "${length}"/>
+            </geometry>
+            <origin xyz = "0 0 0" rpy = "0 0 0"/>
+        </collision>
+        <xacro:wheel m = "1.0" r = "${radius}" h = "${length}"
+                             o_xyz = "0 0 0" o_rpy = "0 0 0"/> -->
     </link>
     <xacro:macro name = "wheel_link" params="prefix">
@@ -77,7 +85,7 @@
         <origin xyz = "0 0 ${radius}" rpy = "0 0 0"/>
     </joint>
-    <joint name = "base_lider_joint" type = "fixed">
+    <joint name = "base_lidar_joint" type = "fixed">
         <parent link = "base_link"/>
-        <child link = "lider_link"/>
+        <child link = "lidar_link"/>
         <origin xyz = "0 0 ${base_height + length / 2.0}" rpy = "0 0 0"/>
     </joint>

File: scr/my_robot_descirption/urdf/my_car.urdf.xacro (robot description, xacro)
@@ -4,3 +4,6 @@
     <xacro:include filename = "mobile_base.xacro"/>
     <xacro:include filename = "mobile_base_gazebo.xacro"/>
+    <xacro:include filename = "gazebo_plugin.xacro"/>
+    <xacro:include filename = "camera_sensor.xacro"/>
+    <xacro:include filename = "lidar.xacro"/>
 </robot>
