Commit message: Add files via upload

File: scr/my_robot_descirption/urdf/camera_sensor.xacro (robot description, xacro)
@@ -4,5 +4,5 @@
     <xacro:property name = "camera_width" value = "0.15"/>
     <xacro:property name = "camera_height" value = "0.08"/>
-    <link name = "camera_lin">
+    <link name = "camera_link">
         <visual>
             <geometry>
@@ -23,5 +23,5 @@
     <joint name  = "camera_link_joint" type = "fixed">
         <parent link = "base_link"/>
-        <child link = "camera_lin"/>
+        <child link = "camera_link"/>
         <origin xyz = "${base_len / 2} 0 ${base_height / 2}" rpy = "0 0 0"/>
         <axis xyz = "0 1 0"/>
